File: kicad/pitubedirect-hat-dip-v1.kicad_pcb (KiCad board)
At the start: 2 copper layers, 58.4 x 63.5 mm, 25 parts, among them P1 CONN_02X20, P2 CONN_02X13, P3 CONN_01X02, P4 CONN_01X03, U1 74LVC245AN, U2 74LVC245AN

Commit message: Added 2nd iteration of PCB design
Change-Id: I13e39ce9abf2ba7743cdcd9543cd2f85d4fc066c
Parts:
- added C8: 15p, Capacitors_ThroughHole:C_Rect_L7_W2_P5, F.Cu at (138.4, 113.7)
- added R13: 470, Discret:R4-5, F.Cu at (135.9, 79.4)
- added REF**: MountingHole_2.7mm_M2.5_Pad, Mounting_Holes:MountingHole_2.7mm_M2.5_Pad, F.Cu at (169.5, 73.2)
- added REF**: MountingHole_2.7mm_M2.5_Pad, Mounting_Holes:MountingHole_2.7mm_M2.5_Pad, F.Cu at (169.5, 131.2)
- added REF**: MountingHole_2.7mm_M2.5_Pad, Mounting_Holes:MountingHole_2.7mm_M2.5_Pad, F.Cu at (120.5, 73.2)
- added REF**: MountingHole_2.7mm_M2.5_Pad, Mounting_Holes:MountingHole_2.7mm_M2.5_Pad, F.Cu at (120.5, 131.2)
- P2: value CONN_02X13 -> CONN_02X20; footprint Pin_Headers:Pin_Header_Straight_2x13 -> Pin_Headers:Pin_Header_Straight_2x20
- R1, R10, R11, R12, R2, R3, R4, R5, R6, R7, R8, R9: footprint Discret:R5 -> Discret:R4-5
- moved P3 69.6 mm to (127.6, 130.8)
- moved C2 57.3 mm to (145.4, 131.4), turned to 90 degrees
- moved P4 10.2 mm to (164.5, 84.5)
- moved C3 3.17 mm to (161.3, 74.9)
- moved P1 1.27 mm to (121.3, 78.1)
- moved C4 0.64 mm to (138.4, 116.2)
- moved C5 0.64 mm to (138.4, 123.8)
- moved C6 0.64 mm to (138.4, 121.3)
- moved C7 0.64 mm to (138.4, 118.7)
- moved R1 0.63 mm to (135.9, 81.9)
- moved R10 0.63 mm to (135.9, 104.8)
- moved R11 0.63 mm to (135.9, 107.3)
- moved R12 0.63 mm to (135.9, 109.9)
- moved R2 0.63 mm to (135.9, 84.5)
- moved R3 0.63 mm to (135.9, 87.0)
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Connections:
- P1 pad 8: /TnTUBE -> Net-(P1-Pad8)
- U2 pad 19: /TnTUBE -> Net-(P1-Pad8)
Routing:
- net +5V: track 101.7 -> 0.00 mm
- net Net-(P1-Pad8): track 0.00 -> 53.1 mm, vias 0 -> 1
- net GND: track 12.3 -> 28.3 mm
- net /TnTUBE: track 60.4 -> 47.0 mm, vias 1 -> 2
- net /RnW: track 37.1 -> 44.7 mm
- net /TPHI2: track 52.2 -> 58.1 mm
- net /PHI2: track 22.3 -> 18.0 mm, vias 1 -> 0
- net /D7: track 21.0 -> 17.3 mm
- net VCC: track 102.5 -> 105.5 mm
- net Net-(P2-Pad8): track 3.81 -> 6.88 mm
- net Net-(P2-Pad10): track 3.81 -> 6.88 mm
- net /TRnW: track 63.7 -> 65.5 mm, vias 0 -> 3
- net Net-(P1-Pad30): track 7.18 -> 8.98 mm
- net Net-(P1-Pad20): track 7.18 -> 8.98 mm
- net Net-(P1-Pad16): track 7.18 -> 8.98 mm
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- added copper zone on F.Cu, net +5V
- added copper zone on F.Cu, net Net-(P2-Pad2)
Other:
- board size 58.4 x 63.5 mm -> 57 x 65 mm
- net class Default: clearance 0.2032 -> 0.254; trace_width 0.2032 -> 0.254
- net class Power: clearance 0.2032 -> 0.254; trace_width 0.3048 -> 0.762
- rule trace_clearance: 0.2032 -> 0.254
- rule trace_min: 0.2032 -> 0.254
- board text added: "PiTubeDirect © 2016 David Banks"
- board text added: "Power Pi fromTube"

Commit message: Added 3rd iteration of PCB design
Change-Id: I3b84f437a23c6d4a3b09af5eeef19cbf285e57d3
Parts:
- P1: footprint Pin_Headers:Pin_Header_Straight_2x20 -> Socket_Strips:Socket_Strip_Angled_2x20
- P2: footprint Pin_Headers:Pin_Header_Straight_2x20 -> Socket_Strips:Socket_Strip_Straight_2x20; moved to B.Cu
- R1, R10, R11, R12, R13, R2, R3, R4, R5, R6, R7, R8, R9: footprint Discret:R4-5 -> Discret:R4
- moved R1 0.64 mm to (136.5, 81.9)
- moved R10 0.64 mm to (136.5, 104.8)
- moved R11 0.64 mm to (136.5, 107.3)
- moved R12 0.64 mm to (136.5, 109.9)
- moved R13 0.64 mm to (136.5, 79.4)
- moved R2 0.64 mm to (136.5, 84.5)
- moved R3 0.64 mm to (136.5, 87.0)
- moved R4 0.64 mm to (136.5, 89.5)
- moved R5 0.64 mm to (136.5, 92.1)
- moved R6 0.64 mm to (136.5, 94.6)
- moved R7 0.64 mm to (136.5, 97.2)
- moved R8 0.64 mm to (136.5, 99.7)
- moved R9 0.64 mm to (136.5, 102.2)
- moved P1 0.64 mm to (121.9, 78.1), turned to 270 degrees
- turned P2 to 270 degrees
Routing:
- net GND: track 28.3 -> 5.39 mm
- net +5V: track 0.00 -> 10.2 mm
- net /TRnW: track 65.5 -> 71.4 mm
- net Net-(P1-Pad32): track 8.98 -> 14.7 mm
- net Net-(P1-Pad30): track 8.98 -> 14.7 mm
- net Net-(P1-Pad28): track 8.98 -> 14.7 mm
- net Net-(P1-Pad26): track 8.98 -> 14.7 mm
- net Net-(P1-Pad24): track 8.98 -> 14.7 mm
- net Net-(P1-Pad22): track 8.98 -> 14.7 mm
- net Net-(P1-Pad20): track 8.98 -> 14.7 mm
- net Net-(P1-Pad18): track 8.98 -> 14.7 mm
- net Net-(P1-Pad16): track 8.98 -> 14.7 mm
- net Net-(P1-Pad14): track 8.98 -> 14.7 mm
- net Net-(P1-Pad12): track 8.98 -> 14.7 mm
- net Net-(P1-Pad10): track 8.98 -> 14.7 mm
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Other:
- outline, holes or cut-outs redrawn
- net class Default: via_dia 0.6858 -> 0.889; via_drill 0.3302 -> 0.381
- net class Power: via_dia 0.6858 -> 0.889; via_drill 0.3302 -> 0.381
- rule via_min_drill: 0.3302 -> 0.381
- rule via_min_size: 0.6858 -> 0.889
- board text added: "Power Pi from Tube"
- board text removed: "Power Pi fromTube"

Commit message: PCB: Added A3
Change-Id: Ifec141e4d1beefc1e0d7cd2525f500dfc024b9c1
Parts:
- added C9: 15p, Capacitors_ThroughHole:C_Rect_L7_W2_P5, F.Cu at (138.4, 120.0)
- added R14: 470, Discret:R4, F.Cu at (136.5, 112.4)
- moved C5 3.81 mm to (138.4, 127.6)
- moved C6 3.81 mm to (138.4, 125.1)
- moved C7 3.81 mm to (138.4, 122.6)
- moved C3 2.29 mm to (162.6, 73.0), turned to 90 degrees
- moved C4 1.27 mm to (138.4, 117.5)
- moved C8 1.27 mm to (138.4, 114.9)
- moved P3 0.63 mm to (127.6, 131.4)
- turned C2 to 180 degrees
Connections:
- P2 pad 29: Net-(P2-Pad29) -> /A3
- U1 pad 15: /TA2 -> /TA3
- U1 pad 16: /TA1 -> /TA2
- U1 pad 17: /TA0 -> /TA1
- U1 pad 18: Net-(U1-Pad18) -> /TA0
- U1 pad 2: Net-(U1-Pad2) -> /A0
- U1 pad 3: /A0 -> /A1
- U1 pad 4: /A1 -> /A2
- U1 pad 5: /A2 -> /A3
Routing:
- net /TA3: track 0.00 -> 22.9 mm
- net /A3: track 0.00 -> 21.5 mm
- net Net-(P1-Pad34): track 0.00 -> 14.7 mm
- net /TA2: track 22.6 -> 28.0 mm
- net /TA1: track 28.8 -> 33.6 mm
- net /TA0: track 34.9 -> 39.2 mm
- net /tnRST: track 45.1 -> 48.1 mm
- net /A2: track 50.8 -> 53.3 mm
- net /A0: track 45.7 -> 48.3 mm
- net /A1: track 55.1 -> 57.7 mm
- net VCC: track 105.5 -> 103.9 mm
- net /TnTUBE: track 47.0 -> 47.5 mm

Commit message: PCB: Updated power connector; changed copyright
Change-Id: Idf6382d1eea538a78420a4489c67f2c6460abd1e
Parts:
- P3: value CONN_01X02 -> CONN_01X03; footprint Pin_Headers:Pin_Header_Straight_1x02 -> Pin_Headers:Pin_Header_Straight_1x03
- moved P3 3.81 mm to (131.4, 131.4), turned to 270 degrees
- moved C4 0.63 mm to (139.1, 117.5)
- moved C5 0.63 mm to (139.1, 127.6)
- moved C6 0.63 mm to (139.1, 125.1)
- moved C7 0.63 mm to (139.1, 122.6)
- moved C8 0.63 mm to (139.1, 114.9)
- moved C9 0.63 mm to (139.1, 120.0)
Connections:
- P3 pad 1: +5V -> GND
Routing:
- net VCC: track 103.9 -> 101.8 mm
- net /tnRST: track 48.1 -> 46.3 mm
- net /TA2: track 28.0 -> 27.1 mm
- net /TA3: track 22.9 -> 22.0 mm
- net /TA1: track 33.6 -> 32.7 mm
- net /TA0: track 39.2 -> 38.3 mm
- net /TnTUBE: track 47.5 -> 46.9 mm
Other:
- board text added: "GND"
- board text added: "Pi +5V"
- board text added: "PiTubeDirect © 2016 Dave, Ed, Rich"
- board text added: "Tube +5V"
- board text removed: "PiTubeDirect © 2016 David Banks"
- board text removed: "Power Pi from Tube"
