File: kicad/pitubedirect-hat-dip-v1.sch (KiCad schematic (older format))
At the start: 25 parts, among them P1 CONN_02X20, P2 CONN_02X13, P3 CONN_01X02, P4 CONN_01X03, U1 74LVC245AN, U2 74LVC245AN

Commit message: Added 2nd iteration of PCB design
Change-Id: I13e39ce9abf2ba7743cdcd9543cd2f85d4fc066c
Parts:
- removed P2: CONN_02X13, Pin_Headers:Pin_Header_Straight_2x13, symbol CONN_02X13
- added C8: 15p, Capacitors_ThroughHole:C_Rect_L7_W2_P5, symbol C_Small
- added P2: CONN_02X20, Pin_Headers:Pin_Header_Straight_2x20, symbol CONN_02X20
- added R13: 470, Discret:R4-5, symbol R
- R1, R10, R11, R12, R2, R3, R4, R5, R6, R7, R8, R9: footprint Discret:R5 -> Discret:R4-5
Connections:
- net A0: now also P2.13 (P13)
- net A1: now also P2.3 (P3)
- net A2: now also P2.5 (P5)
- net D0: now also P2.24 (P24)
- net D1: now also P2.21 (P21)
- net D2: now also P2.19 (P19)
- net D3: now also P2.23 (P23)
- net D4: now also P2.15 (P15)
- net D5: now also P2.16 (P16)
- net D6: now also P2.18 (P18)
- net D7: now also P2.22 (P22)
- net GND: now also C8.2, P2.14 (P14), P2.20 (P20), P2.25 (P25), P2.30 (P30), P2.34 (P34), P2.39 (P39), P2.6 (P6), P2.9 (P9)
- net PHI2: now also P2.26 (P26)
- net RnW: now also P2.12 (P12)
- net TnTUBE: now also C8.1, R13.1; no longer P1.8 (P8), U2.19 (CE)
- net VCC: now also P2.1 (P1), P2.17 (P17)
- net nRST: now also P2.7 (P7)
- net nTUBE: now also P2.11 (P11)
- net at P4.3 (P3): now also P2.10 (P10)
- net at P3.2 (P2): now also P2.2 (P2), P2.4 (P4)
- net at P4.2 (P2): now also P2.8 (P8)
- new net: P1.8 (P8), R13.2, U2.19 (CE)
- no-connect marks 7 -> 20
Other:
- moved on the sheet: R1, R12, R4, R5, R8, R9

Commit message: Added 3rd iteration of PCB design
Change-Id: I3b84f437a23c6d4a3b09af5eeef19cbf285e57d3
Parts:
- P1: footprint Pin_Headers:Pin_Header_Straight_2x20 -> Socket_Strips:Socket_Strip_Angled_2x20
- P2: footprint Pin_Headers:Pin_Header_Straight_2x20 -> Socket_Strips:Socket_Strip_Straight_2x20
- R1, R10, R11, R12, R13, R2, R3, R4, R5, R6, R7, R8, R9: footprint Discret:R4-5 -> Discret:R4
Changed lines of the file:
@@
 F 0 "P1" H 3050 5700 50  0000 C CNN
 F 1 "CONN_02X20" V 3050 4650 50  0000 C CNN
-F 2 "Pin_Headers:Pin_Header_Straight_2x20" H 3050 3700 50  0001 C CNN
+F 2 "Socket_Strips:Socket_Strip_Angled_2x20" H 3050 3700 50  0001 C CNN
 F 3 "" H 3050 3700 50  0000 C CNN
 	1    3050 4650
@@
 F 0 "R9" V 3830 4900 50  0000 C CNN
 F 1 "100" V 3750 4900 50  0000 C CNN
-F 2 "Discret:R4-5" V 3680 4900 50  0001 C CNN
+F 2 "Discret:R4" V 3680 4900 50  0001 C CNN
 F 3 "" H 3750 4900 50  0000 C CNN
 	1    3750 4900
@@
 F 0 "R8" V 3630 4800 50  0000 C CNN
 F 1 "100" V 3550 4800 50  0000 C CNN
-F 2 "Discret:R4-5" V 3480 4800 50  0001 C CNN
+F 2 "Discret:R4" V 3480 4800 50  0001 C CNN
 F 3 "" H 3550 4800 50  0000 C CNN
 	1    3550 4800
@@
 F 0 "R7" V 3830 4700 50  0000 C CNN
 F 1 "100" V 3750 4700 50  0000 C CNN
-F 2 "Discret:R4-5" V 3680 4700 50  0001 C CNN
+F 2 "Discret:R4" V 3680 4700 50  0001 C CNN
 F 3 "" H 3750 4700 50  0000 C CNN
 	1    3750 4700
@@
 F 0 "R6" V 3630 4600 50  0000 C CNN
 F 1 "100" V 3550 4600 50  0000 C CNN
-F 2 "Discret:R4-5" V 3480 4600 50  0001 C CNN
+F 2 "Discret:R4" V 3480 4600 50  0001 C CNN
 F 3 "" H 3550 4600 50  0000 C CNN
 	1    3550 4600
@@
 F 0 "R5" V 3830 4500 50  0000 C CNN
 F 1 "100" V 3750 4500 50  0000 C CNN
-F 2 "Discret:R4-5" V 3680 4500 50  0001 C CNN
+F 2 "Discret:R4" V 3680 4500 50  0001 C CNN
 F 3 "" H 3750 4500 50  0000 C CNN
 	1    3750 4500
@@
 F 0 "R4" V 3630 4400 50  0000 C CNN
 F 1 "100" V 3550 4400 50  0000 C CNN
-F 2 "Discret:R4-5" V 3480 4400 50  0001 C CNN
+F 2 "Discret:R4" V 3480 4400 50  0001 C CNN
 F 3 "" H 3550 4400 50  0000 C CNN
 	1    3550 4400
@@
 F 0 "R3" V 3830 4300 50  0000 C CNN
 F 1 "100" V 3750 4300 50  0000 C CNN
-F 2 "Discret:R4-5" V 3680 4300 50  0001 C CNN
+F 2 "Discret:R4" V 3680 4300 50  0001 C CNN
 F 3 "" H 3750 4300 50  0000 C CNN
 	1    3750 4300
@@
 F 0 "R2" V 3630 4200 50  0000 C CNN
 F 1 "100" V 3550 4200 50  0000 C CNN
-F 2 "Discret:R4-5" V 3480 4200 50  0001 C CNN
+F 2 "Discret:R4" V 3480 4200 50  0001 C CNN
 F 3 "" H 3550 4200 50  0000 C CNN
 	1    3550 4200
@@
 F 0 "R10" V 3630 5000 50  0000 C CNN
 F 1 "470" V 3550 5000 50  0000 C CNN
-F 2 "Discret:R4-5" V 3480 5000 50  0001 C CNN
+F 2 "Discret:R4" V 3480 5000 50  0001 C CNN
 F 3 "" H 3550 5000 50  0000 C CNN
 	1    3550 5000
@@
 F 0 "R11" V 3830 5100 50  0000 C CNN
 F 1 "470" V 3750 5100 50  0000 C CNN
-F 2 "Discret:R4-5" V 3680 5100 50  0001 C CNN
+F 2 "Discret:R4" V 3680 5100 50  0001 C CNN
 F 3 "" H 3750 5100 50  0000 C CNN
 	1    3750 5100
@@
 F 0 "R12" V 3630 5200 50  0000 C CNN
 F 1 "470" V 3550 5200 50  0000 C CNN
-F 2 "Discret:R4-5" V 3480 5200 50  0001 C CNN
+F 2 "Discret:R4" V 3480 5200 50  0001 C CNN
 F 3 "" H 3550 5200 50  0000 C CNN
 	1    3550 5200
@@
 F 0 "R1" V 3830 4100 50  0000 C CNN
 F 1 "470" V 3750 4100 50  0000 C CNN
-F 2 "Discret:R4-5" V 3680 4100 50  0001 C CNN
+F 2 "Discret:R4" V 3680 4100 50  0001 C CNN
 F 3 "" H 3750 4100 50  0000 C CNN
 	1    3750 4100
@@
 F 0 "R13" V 3630 4000 50  0000 C CNN
 F 1 "470" V 3550 4000 50  0000 C CNN
-F 2 "Discret:R4-5" V 3480 4000 50  0001 C CNN
+F 2 "Discret:R4" V 3480 4000 50  0001 C CNN
 F 3 "" H 3550 4000 50  0000 C CNN
 	1    3550 4000
@@
 F 0 "P2" H 8400 5000 50  0000 C CNN
 F 1 "CONN_02X20" V 8400 3950 50  0000 C CNN
-F 2 "Pin_Headers:Pin_Header_Straight_2x20" H 8400 3000 50  0001 C CNN
+F 2 "Socket_Strips:Socket_Strip_Straight_2x20" H 8400 3000 50  0001 C CNN
 F 3 "" H 8400 3000 50  0000 C CNN
 	1    8400 3950

Commit message: PCB: Added A3
Change-Id: Ifec141e4d1beefc1e0d7cd2525f500dfc024b9c1
Parts:
- added C9: 15p, Capacitors_ThroughHole:C_Rect_L7_W2_P5, symbol C_Small
- added R14: 470, Discret:R4, symbol R
Connections:
- net A0: now also U1.2 (A0); no longer U1.3 (A1)
- net A1: now also U1.3 (A1); no longer U1.4 (A2)
- net A2: now also U1.4 (A2); no longer U1.5 (A3)
- net GND: now also C9.2
- net TA0: now also U1.18 (B0); no longer U1.17 (B1)
- net TA1: now also U1.17 (B1); no longer U1.16 (B2)
- net TA2: now also U1.16 (B2); no longer U1.15 (B3)
- net at P1.34 (P34): now also R14.2
- net A3: now reaches P2.29 (P29)
- net A3: now also U1.5 (A3)
- new net TA3: C9.1, R14.1, U1.15 (B3)
- no-connect marks 20 -> 14
Other:
- moved on the sheet: U1

Commit message: PCB: Updated power connector; changed copyright
Change-Id: Idf6382d1eea538a78420a4489c67f2c6460abd1e
Parts:
- removed P3: CONN_01X02, Pin_Headers:Pin_Header_Straight_1x02, symbol CONN_01X02
- added P3: CONN_01X03, Pin_Headers:Pin_Header_Straight_1x03, symbol CONN_01X03
Connections:
- net +5V: now also P3.3 (P3)
- net GND: now also P3.1 (P1)
- net at P2.2 (P2), P2.4 (P4): now also P3.2 (P2)
Changed lines of the file:
@@
-$EndComp
-$Comp
-L CONN_01X02 P3
-U 1 1 574305E2
-P 8400 2500
-F 0 "P3" H 8400 2650 50  0000 C CNN
-F 1 "CONN_01X02" V 8500 2500 50  0000 C CNN
-F 2 "Pin_Headers:Pin_Header_Straight_1x02" H 8400 2500 50  0001 C CNN
-F 3 "" H 8400 2500 50  0000 C CNN
-	1    8400 2500
-	-1   0    0    -1
 $EndComp
 $Comp
 L +5V #PWR07
 U 1 1 57430BA3
-P 8750 2300
-F 0 "#PWR07" H 8750 2150 50  0001 C CNN
-F 1 "+5V" H 8750 2440 50  0000 C CNN
-F 2 "" H 8750 2300 50  0000 C CNN
-F 3 "" H 8750 2300 50  0000 C CNN
-	1    8750 2300
+P 8550 2250
+F 0 "#PWR07" H 8550 2100 50  0001 C CNN
+F 1 "+5V" H 8550 2390 50  0000 C CNN
+F 2 "" H 8550 2250 50  0000 C CNN
+F 3 "" H 8550 2250 50  0000 C CNN
+	1    8550 2250
 	1    0    0    -1
 $EndComp
@@
 	2550 1800 2550 1900
 Wire Wire Line
-	8750 2450 8750 2300
-Wire Wire Line
-	8600 2450 8750 2450
+	8550 2350 8550 2250
+Wire Wire Line
+	8450 2350 8550 2350
 Wire Wire Line
 	2050 2200 2050 2400
@@
 Connection ~ 8750 3000
 Wire Wire Line
-	8750 2550 8600 2550
+	8450 2450 8750 2450
 Wire Wire Line
 	8750 3000 8650 3000
 Wire Wire Line
-	8750 2550 8750 3100
+	8750 2450 8750 3100
 Wire Wire Line
 	8750 3100 8650 3100
@@
 Text Label 6950 2900 0    60   ~ 0
 A3
+$Comp
+L CONN_01X03 P3
+U 1 1 5776A5E5
+P 8250 2450
+F 0 "P3" H 8250 2650 50  0000 C CNN
+F 1 "CONN_01X03" V 8350 2450 50  0000 C CNN
+F 2 "Pin_Headers:Pin_Header_Straight_1x03" H 8250 2450 50  0001 C CNN
+F 3 "" H 8250 2450 50  0000 C CNN
+	1    8250 2450
+	-1   0    0    1
+$EndComp
+$Comp
+L GND #PWR015
+U 1 1 5776AB51
+P 8550 2650
+F 0 "#PWR015" H 8550 2400 50  0001 C CNN
+F 1 "GND" H 8550 2500 50  0000 C CNN
+F 2 "" H 8550 2650 50  0000 C CNN
+F 3 "" H 8550 2650 50  0000 C CNN
+	1    8550 2650
+	1    0    0    -1
+$EndComp
+Wire Wire Line
+	8450 2550 8550 2550
+Wire Wire Line
+	8550 2550 8550 2650
 $EndSCHEMATC
